File: Hardware/smartlockcc.kicad_sch (KiCad schematic)
At the start: 26 parts, among them J1 USB4085-GF-A_REVB, J2 Conn_01x04_Pin, J3 Conn_01x02_Socket, J4 Conn_01x02_Socket, J5 Conn_01x05, M1 Motor_Servo, P1 RFID-RC522-MODULE, Q2 Q_NMOS_GSD, U1 ESP32-C3-WROOM-02, U2 AZ1117-3.3

Commit message: Cleanup and pictures added
Other:
- note added: "+3V3 LED"
- note added: "ESP32 Decoupling"
- note added: "Free GPIOs Conn."
- note added: "Power transistor"
- note added: "RFID Connector"
- note added: "UART Debug Conn."
- note removed: "Power LED"
- note removed: "To USB-UART board"
- title: (none) -> SmartLockCC
- moved on the sheet: C1, C2, C3, J2, J3, J4, J5, M1, P1, Q2, R1, R4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
